Commit message: Updated training logic, gait reward functions and environment file to track velocity and success and failed episodes

File: dodobot_v3/urdf/dodobot_v3_simple.urdf (robot description, URDF)
Before this commit: robot dodobot_v3, 10 links, 9 joints
Links:
- link body_link: geometry collision box size=0.21 0.29 0.23; visual mesh filename=/home/aaron/dodo_rl/dodobot_v3/meshes/body_link.STL
- link left_link_1: geometry visual mesh filename=/home/aaron/dodo_rl/dodobot_v3/meshes/left_link_1.STL
- link left_link_2: geometry collision cylinder length=0.18 radius=0.03; visual mesh filename=/home/aaron/dodo_rl/dodobot_v3/meshes/left_link_2.STL
- link left_link_3: geometry collision cylinder length=0.14 radius=0.03; visual mesh filename=/home/aaron/dodo_rl/dodobot_v3/meshes/left_link_3.STL
- link left_link_4: geometry collision box size=0.095 0.036 0.0615; visual mesh filename=/home/aaron/dodo_rl/dodobot_v3/meshes/left_link_4.STL
- link right_link_1: geometry visual mesh filename=/home/aaron/dodo_rl/dodobot_v3/meshes/right_link_1.STL
- link right_link_2: geometry collision cylinder length=0.18 radius=0.03; visual mesh filename=/home/aaron/dodo_rl/dodobot_v3/meshes/right_link_2.STL
- link right_link_3: geometry collision cylinder length=0.14 radius=0.03; visual mesh filename=/home/aaron/dodo_rl/dodobot_v3/meshes/right_link_3.STL
- link right_link_4: geometry collision box size=0.095 0.036 0.0615; visual mesh filename=/home/aaron/dodo_rl/dodobot_v3/meshes/right_link_4.STL
